File: lab4/exercise1/exercise1.kicad_sch (KiCad schematic)
At the start: 6 parts, among them J1 9 V, SW1 

Commit message: panda
Parts:
- C1: footprint (none) -> Capacitor_THT:C_Radial_D5.0mm_H5.0mm_P2.00mm
- D1: footprint (none) -> LED_THT:LED_D5.0mm
- J1: footprint (none) -> Connector_JST:JST_PH_B2B-PH-K_1x02_P2.00mm_Vertical
- R1, R2: footprint (none) -> Resistor_THT:R_Axial_DIN0516_L15.5mm_D5.0mm_P20.32mm_Horizontal
- SW1: footprint (none) -> Button_Switch_THT:SW_E-Switch_EG1224_SPDT_Angled
Changed lines of the file:
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@@
     )
     (property "Value" " " (id 1) (at 139.7 55.88 0))
-    (property "Footprint" "" (id 2) (at 139.7 60.96 0)
+    (property "Footprint" "Button_Switch_THT:SW_E-Switch_EG1224_SPDT_Angled" (id 2) (at 139.7 60.96 0)
       (effects (font (size 1.27 1.27)) hide)
     )
@@
       (effects (font (size 1.27 1.27)) (justify left))
     )
-    (property "Footprint" "" (id 2) (at 177.292 73.66 90)
+    (property "Footprint" "Resistor_THT:R_Axial_DIN0516_L15.5mm_D5.0mm_P20.32mm_Horizontal" (id 2) (at 177.292 73.66 90)
       (effects (font (size 1.27 1.27)) hide)
     )
@@
     (property "Reference" "J1" (id 0) (at 120.65 95.25 0))
     (property "Value" "9 V" (id 1) (at 120.65 97.79 0))
-    (property "Footprint" "" (id 2) (at 113.03 96.52 0)
+    (property "Footprint" "Connector_JST:JST_PH_B2B-PH-K_1x02_P2.00mm_Vertical" (id 2) (at 113.03 96.52 0)
       (effects (font (size 1.27 1.27)) hide)
     )
@@
     (property "Reference" "R2" (id 0) (at 125.73 63.5 90))
     (property "Value" "2.2 kΩ" (id 1) (at 125.73 66.04 90))
-    (property "Footprint" "" (id 2) (at 125.73 62.738 90)
+    (property "Footprint" "Resistor_THT:R_Axial_DIN0516_L15.5mm_D5.0mm_P20.32mm_Horizontal" (id 2) (at 125.73 62.738 90)
       (effects (font (size 1.27 1.27)) hide)
     )
@@
       (effects (font (size 1.27 1.27)) (justify right))
     )
-    (property "Footprint" "" (id 2) (at 179.07 97.79 0)
+    (property "Footprint" "LED_THT:LED_D5.0mm" (id 2) (at 179.07 97.79 0)
       (effects (font (size 1.27 1.27)) hide)
     )
@@
       (effects (font (size 1.27 1.27)) (justify left))
     )
-    (property "Footprint" "" (id 2) (at 150.8252 90.17 0)
+    (property "Footprint" "Capacitor_THT:C_Radial_D5.0mm_H5.0mm_P2.00mm" (id 2) (at 150.8252 90.17 0)
       (effects (font (size 1.27 1.27)) hide)
     )
@@
   (symbol_instances
     (path "/ee0fca32-d38f-4a61-8c0b-9943a05499ee"
-      (reference "C1") (unit 1) (value "4.7 μF") (footprint "")
+      (reference "C1") (unit 1) (value "4.7 μF") (footprint "Capacitor_THT:C_Radial_D5.0mm_H5.0mm_P2.00mm")
     )
     (path "/e870f6ea-9264-4d5f-befb-7f2c555a0825"
-      (reference "D1") (unit 1) (value "LED") (footprint "")
+      (reference "D1") (unit 1) (value "LED") (footprint "LED_THT:LED_D5.0mm")
     )
     (path "/6cc87d7e-5229-49cd-8815-ff98a193f10f"
-      (reference "J1") (unit 1) (value "9 V") (footprint "")
+      (reference "J1") (unit 1) (value "9 V") (footprint "Connector_JST:JST_PH_B2B-PH-K_1x02_P2.00mm_Vertical")
     )
     (path "/11fa7c8b-51d6-476b-a0c4-ae05e79874bf"
-      (reference "R1") (unit 1) (value "20 kΩ") (footprint "")
+      (reference "R1") (unit 1) (value "20 kΩ") (footprint "Resistor_THT:R_Axial_DIN0516_L15.5mm_D5.0mm_P20.32mm_Horizontal")
     )
     (path "/8207be84-b6ca-4eac-be40-fcc4a71377a3"
-      (reference "R2") (unit 1) (value "2.2 kΩ") (footprint "")
+      (reference "R2") (unit 1) (value "2.2 kΩ") (footprint "Resistor_THT:R_Axial_DIN0516_L15.5mm_D5.0mm_P20.32mm_Horizontal")
     )
     (path "/05247773-773a-4381-8976-36fcb76884d4"
-      (reference "SW1") (unit 1) (value " ") (footprint "")
+      (reference "SW1") (unit 1) (value " ") (footprint "Button_Switch_THT:SW_E-Switch_EG1224_SPDT_Angled")
     )
   )
