File: lab4/exercise1/exercise1.kicad_pcb (KiCad board)
At the start: 2 copper layers, 119.4 x 78.7 mm, 6 parts, among them J1 9 V, SW1 

Commit message: panda
Routing:
- added copper zone on F.Cu, net Net-(J1-Pad1)
Changed lines of the file:
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@@
   (segment (start 118.3 48.26) (end 117.125 47.085) (width 0.25) (layer "F.Cu") (net 5))
   (segment (start 112.638299 48.26) (end 93.98 48.26) (width 0.25) (layer "F.Cu") (net 5))
+  (zone (net 4) (net_name "Net-(J1-Pad1)") (layer "F.Cu") (hatch edge 0.508)
+    (connect_pads (clearance 0.508))
+    (min_thickness 0.254) (filled_areas_thickness no)
+    (fill yes (thermal_gap 0.508) (thermal_bridge_width 0.508))
+    (polygon
+      (pts
+        (xy 175.26 106.68)
+        (xy 71.12 106.68)
+        (xy 71.12 43.18)
+        (xy 175.26 43.18)
+      )
+    )
+  )
 )
