File: lab4/exercise2/exercise2.kicad_pcb (KiCad board)
At the start: 2 copper layers, 68.6 x 58.4 mm, 10 parts, among them J1 , U1 

Commit message: panda
Parts:
- moved R4 11.9 mm to (149.9, 83.8)
- moved D1 7.62 mm to (149.9, 71.1)
- moved D2 3.79 mm to (154.2, 104.7)
- moved C1 2.54 mm to (111.8, 104.1)
- moved R3 2.54 mm to (154.9, 78.7)
Routing:
- net /pin_3: track 48.6 -> 36.7 mm
- net +9V: track 83.2 -> 74.1 mm
- net Net-(D2-Pad2): track 14.1 -> 22.9 mm
- net GND: track 100.9 -> 94.6 mm
- net /pin_2: track 90.1 -> 92.6 mm
- net Net-(D1-Pad1): track 7.24 -> 8.11 mm
- added copper zone on F.Cu, net (none)
